File: Board/Eagle/SnowFlake.brd (EAGLE design)
At the start: 69.1 x 79.8 mm, 51 parts, among them IC1 ATSAMD20E-TQFP32, J2 CON-SNOWF-IN, J3 CON-SNOWF-OUT

Commit message: Fixing the capacitor value in the schema from 10µF to 1µF.
Parts:
- C4, C5: value 10µF -> 1µF
Changed lines of the file:
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@@
 <?xml version="1.0" encoding="utf-8"?>
 <!DOCTYPE eagle SYSTEM "eagle.dtd">
-<eagle version="8.3.2">
+<eagle version="8.5.1">
 <drawing>
 <settings>
-<setting alwaysvectorfont="no"/>
+<setting alwaysvectorfont="yes"/>
 <setting verticaltext="up"/>
 </settings>
@@
 <param name="dpMaxLengthDifference" value="10mm"/>
 <param name="dpGapFactor" value="2.5"/>
-<param name="checkGrid" value="0"/>
 <param name="checkAngle" value="0"/>
 <param name="checkFont" value="1"/>
 <param name="checkRestrict" value="1"/>
+<param name="checkStop" value="0"/>
+<param name="checkValues" value="0"/>
 <param name="useDiameter" value="13"/>
 <param name="maxErrors" value="50"/>
@@
 <element name="J2" library="lucky-resistor" library_urn="urn:adsk.eagle:library:481313" package="CON-PADS-3XWIRE-B" package3d_urn="urn:adsk.eagle:package:493621/2" value="CON-SNOWF-IN" x="40" y="72.75" rot="MR0"/>
 <element name="J3" library="lucky-resistor" library_urn="urn:adsk.eagle:library:481313" package="CON-PADS-3XWIRE-T" package3d_urn="urn:adsk.eagle:package:493620/2" value="CON-SNOWF-OUT" x="40" y="7.55" rot="MR0"/>
-<element name="C4" library="lucky-resistor" library_urn="urn:adsk.eagle:library:481313" package="CAPACITOR-0805-MURATA-GRM-21" package3d_urn="urn:adsk.eagle:package:481485/1" value="10µF" x="24" y="52" smashed="yes" rot="MR0">
+<element name="C4" library="lucky-resistor" library_urn="urn:adsk.eagle:library:481313" package="CAPACITOR-0805-MURATA-GRM-21" package3d_urn="urn:adsk.eagle:package:481485/1" value="1µF" x="24" y="52" smashed="yes" rot="MR0">
 <attribute name="NAME" x="23.5" y="49.65" size="1.016" layer="26" rot="MR0" align="bottom-center"/>
 <attribute name="VALUE" x="24" y="51" size="1.016" layer="28" rot="MR0" align="top-center"/>
 </element>
-<element name="C5" library="lucky-resistor" library_urn="urn:adsk.eagle:library:481313" package="CAPACITOR-0805-MURATA-GRM-21" package3d_urn="urn:adsk.eagle:package:481485/1" value="10µF" x="56" y="29" smashed="yes" rot="MR180">
+<element name="C5" library="lucky-resistor" library_urn="urn:adsk.eagle:library:481313" package="CAPACITOR-0805-MURATA-GRM-21" package3d_urn="urn:adsk.eagle:package:481485/1" value="1µF" x="56" y="29" smashed="yes" rot="MR180">
 <attribute name="NAME" x="56" y="27.7" size="1.016" layer="26" rot="MR180" align="bottom-center"/>
 <attribute name="VALUE" x="56" y="30" size="1.016" layer="28" rot="MR180" align="top-center"/>
